File: InfoAmazonia.sch (EAGLE design)
At the start: 83 parts, among them IC1 LM2662, IC10 4053D, IC11 74HC4051, IC12 4053D, IC13 4053D, IC2 ADAFRUIT FONA, IC3 MIC29302AWD, IC4 4050D, IC5 TL032C, IC6 CA3140AM Z, IC7 TL081BCDG4, IC8 SHT20, IC9 NE555, J1 BNCPTH, J2 BNCPTH, J3 BNCPTH, U1 ARDUINO-MEGAPRO, U2 MPL3115A2, U3 USD-SOCKETNEW, U4 ALS-PT19

Commit message: - Faltando somente distribuicao do +3V3 e decidir se a interrupcao do sensor de pressao fica
Connections:
- removed net A: IC11.A
- removed net B: IC11.B
- removed net C: IC11.C
- new net SELECT_A: IC11.A, U1.42
- new net SELECT_B: IC11.B, U1.43
- new net SELECT_C: IC11.C, U1.40
- net 1_SENSOR_EN: now also U1.A5
- net 2_SENSOR_EN: now also U1.A6
- net 3_SENSOR_EN: now also U1.A7
- net D44: now also IC11.Y5
- net D45: now also IC11.Y7
Other:
- moved on the sheet: C33
Changed lines of the file:
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@@
 <sheet>
 <plain>
-<wire x1="256.54" y1="-60.96" x2="256.54" y2="-127" width="0.1524" layer="94"/>
-<wire x1="256.54" y1="-127" x2="386.08" y2="-127" width="0.1524" layer="94"/>
+<wire x1="254" y1="-60.96" x2="254" y2="-127" width="0.1524" layer="94"/>
+<wire x1="254" y1="-127" x2="386.08" y2="-127" width="0.1524" layer="94"/>
 <wire x1="386.08" y1="-127" x2="386.08" y2="-60.96" width="0.1524" layer="94"/>
-<wire x1="386.08" y1="-60.96" x2="256.54" y2="-60.96" width="0.1524" layer="94"/>
-<wire x1="256.54" y1="0" x2="256.54" y2="-58.42" width="0.1524" layer="94"/>
-<wire x1="256.54" y1="-58.42" x2="386.08" y2="-58.42" width="0.1524" layer="94"/>
+<wire x1="386.08" y1="-60.96" x2="254" y2="-60.96" width="0.1524" layer="94"/>
+<wire x1="254" y1="0" x2="254" y2="-58.42" width="0.1524" layer="94"/>
+<wire x1="254" y1="-58.42" x2="386.08" y2="-58.42" width="0.1524" layer="94"/>
 <wire x1="386.08" y1="-58.42" x2="386.08" y2="0" width="0.1524" layer="94"/>
-<wire x1="386.08" y1="0" x2="256.54" y2="0" width="0.1524" layer="94"/>
+<wire x1="386.08" y1="0" x2="254" y2="0" width="0.1524" layer="94"/>
 <text x="302.26" y="-5.08" size="3.81" layer="94" ratio="10">SENSOR ORP</text>
 <text x="307.34" y="-66.04" size="3.81" layer="94" ratio="10">SENSOR PH</text>
@@
 <text x="53.34" y="-93.98" size="3.81" layer="94" ratio="10">GERADOR +BAT</text>
 <wire x1="116.84" y1="-30.48" x2="116.84" y2="-86.36" width="0.1524" layer="94"/>
-<wire x1="116.84" y1="-30.48" x2="246.38" y2="-30.48" width="0.1524" layer="94"/>
-<wire x1="246.38" y1="-30.48" x2="246.38" y2="-86.36" width="0.1524" layer="94"/>
-<wire x1="246.38" y1="-86.36" x2="116.84" y2="-86.36" width="0.1524" layer="94"/>
+<wire x1="116.84" y1="-30.48" x2="251.46" y2="-30.48" width="0.1524" layer="94"/>
+<wire x1="251.46" y1="-30.48" x2="251.46" y2="-86.36" width="0.1524" layer="94"/>
+<wire x1="251.46" y1="-86.36" x2="116.84" y2="-86.36" width="0.1524" layer="94"/>
 <wire x1="33.02" y1="-127" x2="-38.1" y2="-127" width="0.1524" layer="94"/>
 <wire x1="-38.1" y1="-127" x2="-38.1" y2="-88.9" width="0.1524" layer="94"/>
@@
 <text x="231.14" y="-93.98" size="3.81" layer="94" ratio="10">LUZ</text>
 <wire x1="220.98" y1="-127" x2="220.98" y2="-88.9" width="0.1524" layer="94"/>
-<wire x1="223.52" y1="-88.9" x2="246.38" y2="-88.9" width="0.1524" layer="94"/>
-<wire x1="246.38" y1="-88.9" x2="246.38" y2="-127" width="0.1524" layer="94"/>
-<wire x1="246.38" y1="-127" x2="223.52" y2="-127" width="0.1524" layer="94"/>
+<wire x1="223.52" y1="-88.9" x2="251.46" y2="-88.9" width="0.1524" layer="94"/>
+<wire x1="251.46" y1="-88.9" x2="251.46" y2="-127" width="0.1524" layer="94"/>
+<wire x1="251.46" y1="-127" x2="223.52" y2="-127" width="0.1524" layer="94"/>
 <text x="167.64" y="-35.56" size="3.81" layer="94" ratio="10">CARTÃO SD</text>
 <text x="281.94" y="53.34" size="3.81" layer="94" ratio="10">SENSOR EC</text>
-<wire x1="256.54" y1="2.54" x2="256.54" y2="58.42" width="0.1524" layer="94"/>
-<wire x1="256.54" y1="58.42" x2="386.08" y2="58.42" width="0.1524" layer="94"/>
+<wire x1="254" y1="2.54" x2="254" y2="58.42" width="0.1524" layer="94"/>
+<wire x1="254" y1="58.42" x2="386.08" y2="58.42" width="0.1524" layer="94"/>
 <wire x1="386.08" y1="58.42" x2="386.08" y2="2.54" width="0.1524" layer="94"/>
-<wire x1="386.08" y1="2.54" x2="256.54" y2="2.54" width="0.1524" layer="94"/>
+<wire x1="386.08" y1="2.54" x2="254" y2="2.54" width="0.1524" layer="94"/>
 <wire x1="-38.1" y1="-86.36" x2="-38.1" y2="-30.48" width="0.1524" layer="94"/>
 <wire x1="33.02" y1="-86.36" x2="33.02" y2="-30.48" width="0.1524" layer="94"/>
@@
 <attribute name="VALUE" x="38.1" y="-5.08" size="1.778" layer="96" rot="R180"/>
 </instance>
-<instance part="GND50" gate="1" x="66.04" y="-22.86" smashed="yes">
-<attribute name="VALUE" x="63.5" y="-25.4" size="1.778" layer="96"/>
-</instance>
-<instance part="C33" gate="G$1" x="76.2" y="-15.24" smashed="yes">
-<attribute name="NAME" x="77.724" y="-14.859" size="1.778" layer="95"/>
-<attribute name="VALUE" x="77.724" y="-19.939" size="1.778" layer="96"/>
-</instance>
-<instance part="P+10" gate="1" x="76.2" y="-10.16" smashed="yes">
-<attribute name="VALUE" x="78.74" y="-7.62" size="1.778" layer="96" rot="R180"/>
-</instance>
-<instance part="GND49" gate="1" x="76.2" y="-22.86" smashed="yes">
+<instance part="GND50" gate="1" x="76.2" y="-22.86" smashed="yes">
 <attribute name="VALUE" x="73.66" y="-25.4" size="1.778" layer="96"/>
+</instance>
+<instance part="C33" gate="G$1" x="83.82" y="-15.24" smashed="yes">
+<attribute name="NAME" x="85.344" y="-14.859" size="1.778" layer="95"/>
+<attribute name="VALUE" x="85.344" y="-19.939" size="1.778" layer="96"/>
+</instance>
+<instance part="P+10" gate="1" x="83.82" y="-10.16" smashed="yes">
+<attribute name="VALUE" x="86.36" y="-7.62" size="1.778" layer="96" rot="R180"/>
+</instance>
+<instance part="GND49" gate="1" x="83.82" y="-22.86" smashed="yes">
+<attribute name="VALUE" x="81.28" y="-25.4" size="1.778" layer="96"/>
 </instance>
 <instance part="R15" gate="G$1" x="12.7" y="96.52" smashed="yes" rot="R90">
@@
 <pinref part="IC11" gate="A" pin="/E"/>
 <pinref part="GND50" gate="1" pin="GND"/>
-<wire x1="58.42" y1="-10.16" x2="66.04" y2="-10.16" width="0.1524" layer="91"/>
-<wire x1="66.04" y1="-10.16" x2="66.04" y2="-20.32" width="0.1524" layer="91"/>
+<wire x1="58.42" y1="-10.16" x2="76.2" y2="-10.16" width="0.1524" layer="91"/>
+<wire x1="76.2" y1="-10.16" x2="76.2" y2="-20.32" width="0.1524" layer="91"/>
 </segment>
 <segment>
@@
 </segment>
 </net>
-<net name="A" class="0">
+<net name="SELECT_A" class="0">
 <segment>
 <pinref part="IC11" gate="A" pin="A"/>
@@
 <label x="60.96" y="-12.7" size="1.778" layer="95"/>
 </segment>
-</net>
-<net name="B" class="0">
+<segment>
+<pinref part="U1" gate="G$1" pin="42"/>
+<wire x1="-2.54" y1="12.7" x2="7.62" y2="12.7" width="0.1524" layer="91"/>
+<label x="0" y="12.7" size="1.778" layer="95"/>
+</segment>
+</net>
+<net name="SELECT_B" class="0">
 <segment>
 <pinref part="IC11" gate="A" pin="B"/>
@@
 <label x="60.96" y="-15.24" size="1.778" layer="95"/>
 </segment>
-</net>
-<net name="C" class="0">
+<segment>
+<pinref part="U1" gate="G$1" pin="43"/>
+<wire x1="-2.54" y1="10.16" x2="7.62" y2="10.16" width="0.1524" layer="91"/>
+<label x="0" y="10.16" size="1.778" layer="95"/>
+</segment>
+</net>
+<net name="SELECT_C" class="0">
 <segment>
 <pinref part="IC11" gate="A" pin="C"/>
@@
 <label x="60.96" y="-17.78" size="1.778" layer="95"/>
 </segment>
+<segment>
+<pinref part="U1" gate="G$1" pin="40"/>
+<wire x1="-2.54" y1="17.78" x2="7.62" y2="17.78" width="0.1524" layer="91"/>
+<label x="0" y="17.78" size="1.778" layer="95"/>
+</segment>
 </net>
 <net name="D44" class="0">
@@
 </segment>
 <segment>
-<label x="78.74" y="-5.08" size="1.778" layer="95"/>
-<wire x1="86.36" y1="-5.08" x2="78.74" y2="-5.08" width="0.1524" layer="91"/>
+<pinref part="IC11" gate="A" pin="Y5"/>
+<wire x1="58.42" y1="0" x2="73.66" y2="0" width="0.1524" layer="91"/>
+<label x="63.5" y="0" size="1.778" layer="95"/>
 </segment>
 </net>
@@
 </segment>
 <segment>
-<label x="78.74" y="2.54" size="1.778" layer="95"/>
-<wire x1="86.36" y1="2.54" x2="78.74" y2="2.54" width="0.1524" layer="91"/>
+<pinref part="IC11" gate="A" pin="Y7"/>
+<wire x1="58.42" y1="-5.08" x2="73.66" y2="-5.08" width="0.1524" layer="91"/>
+<label x="63.5" y="-5.08" size="1.778" layer="95"/>
 </segment>
 </net>
@@
 <label x="172.72" y="86.36" size="1.778" layer="95"/>
 </segment>
+<segment>
+<pinref part="U1" gate="G$1" pin="A5"/>
+<wire x1="-43.18" y1="55.88" x2="-66.04" y2="55.88" width="0.1524" layer="91"/>
+<label x="-66.04" y="55.88" size="1.778" layer="95"/>
+</segment>
 </net>
 <net name="2_SENSOR_EN" class="0">
@@
 <label x="172.72" y="38.1" size="1.778" layer="95"/>
 </segment>
+<segment>
+<pinref part="U1" gate="G$1" pin="A6"/>
+<wire x1="-43.18" y1="53.34" x2="-66.04" y2="53.34" width="0.1524" layer="91"/>
+<label x="-66.04" y="53.34" size="1.778" layer="95"/>
+</segment>
 </net>
 <net name="3_SENSOR_EN" class="0">
@@
 <wire x1="162.56" y1="-12.7" x2="170.18" y2="-12.7" width="0.1524" layer="91"/>
 </segment>
-</net>
+<segment>
+<pinref part="U1" gate="G$1" pin="A7"/>
+<wire x1="-43.18" y1="50.8" x2="-66.04" y2="50.8" width="0.1524" layer="91"/>
+<label x="-66.04" y="50.8" size="1.778" layer="95"/>
+</segment>
+</net>

Commit message: - Roteamento terminado, pendendo revisão
Parts:
- removed MD7, MD8: INFO-AMAZONIA-MODULE, InfoAmazonia:INFO-AMAZONIA-MODULE
- added MD2, MD3: INFO-AMAZONIA-MODULE, InfoAmazonia:INFO-AMAZONIA-MODULE
- C12: value 10uF -> 220uF; device InfoAmazonia:C-EUC0603 -> InfoAmazonia:CPOL-EUUD6,3-5,8
- C17, C18, C27, C29: value 10uF -> 100nF
- C19: value 2.2nF -> 10uF
- C20: value 1uF -> 100nF
- C28: value 100nF -> 2.2nF
- C30: value 100nF -> 1uF
- C32, C34, C36, C38: value 100nF -> 10uF
- C6: value 220uF -> 100nF; device InfoAmazonia:CPOL-EUUD6,3-5,8 -> InfoAmazonia:C-EUC0603
- IC1: value LM2662 -> ADAFRUIT FONA; device InfoAmazonia:LM2662 -> InfoAmazonia:ADAFRUIT_FONA
- IC10: value 4053D -> TL032C; device InfoAmazonia:4053D -> InfoAmazonia:AMPOP_2R
- IC11: value 74HC4051 -> NE555; device InfoAmazonia:4051D -> InfoAmazonia:NE555
- IC12: value 4053D -> CA3140AM Z; device InfoAmazonia:4053D -> InfoAmazonia:AMPOP
- IC13: value 4053D -> TL081BCDG4; device InfoAmazonia:4053D -> InfoAmazonia:AMPOP
- IC2: value ADAFRUIT FONA -> LM2662; device InfoAmazonia:ADAFRUIT_FONA -> InfoAmazonia:LM2662
- IC3: value MIC29302AWD -> 74HC4051; device InfoAmazonia:MIC29XXX -> InfoAmazonia:4051D
- IC4: value 4050D -> MIC29302AWD; device InfoAmazonia:4050D -> InfoAmazonia:MIC29XXX
- IC5: value TL032C -> 4050D; device InfoAmazonia:AMPOP_2R -> InfoAmazonia:4050D
- IC6: value CA3140AM Z -> 4053D; device InfoAmazonia:AMPOP -> InfoAmazonia:4053D
- IC7: value TL081BCDG4 -> 4053D; device InfoAmazonia:AMPOP -> InfoAmazonia:4053D
- IC8: value SHT20 -> 4053D; device InfoAmazonia:SHT2X -> InfoAmazonia:4053D
- IC9: value NE555 -> SHT20; device InfoAmazonia:NE555 -> InfoAmazonia:SHT2X
- JP1: value (none) -> ANALOG
- JP2: value (none) -> SERIAL
- JP3: value (none) -> I2C
- JP4: value (none) -> PWM
- R1: value 43k -> 10k
- R10: value 75k -> 5k; device InfoAmazonia:R-EU_R0603 -> InfoAmazonia:RTRIM329W
- R11: value 30k -> 2k2
- R13, R15: value 10k -> 30k
- R14: value 10k -> 75k
- R2: value 100k -> 10k
- R3: value 4M7 -> 43
- R4: value 1k -> 100
- R5: value 5k -> 10k; device InfoAmazonia:RTRIM329W -> InfoAmazonia:R-EU_R0603
- R6: value 2k2 -> 4M7
- R8: value 30k -> 1k
- renumbered JP14 to JP1, JP15 to JP3, JP16 to JP2, JP17 to JP4
Connections:
- removed net INT1: U1.18(TX1), U2.INT1
- removed net INT2: U1.19(RX1), U2.INT2
- net +12V: now also IC4.IN; no longer IC3.IN
- net +3V3: now also C16.1, C17.1, C19.1, C20.1, IC5P.VDD, IC9.VCC; no longer C11.1, C13.1, C28.1, C29.1, IC4P.VDD, IC8.VCC
- net +5V: now also C10.1, C11.1, C6.1, C9.1, IC1.VIO, IC2.V+, IC3.VCC, IC6.VCC, IC6.X, IC7.VCC, IC7.X, IC8.VCC, IC8.X, R1.2, R2.2; no longer C33.1, C34.1, C36.1, C38.1, IC1.V+, IC10.VCC, IC10.X, IC11.VCC, IC12.VCC, IC12.X, IC13.VCC, IC13.X, IC2.VIO, R14.2, R15.2
- net +VBAT: now also C12.+, IC1.BAT, IC4.OUT, R4.1; no longer C6.+, IC2.BAT, IC3.OUT, R2.1
- net +VEC: now also C21.1, IC11./RES, IC11.VCC+, MD5.+5V; no longer C31.1, IC9./RES, IC9.VCC+, MD6.+5V
- net +VORP: now also C31.1, C32.1, IC10P.V+, MD6.+5V; no longer C14.1, C17.1, IC5P.V+, MD5.+5V
- net +VPH: now also C33.1, C34.1, IC12.+VS, IC13.+VS; no longer C12.1, C9.1, IC6.+VS, IC7.+VS
- net -5V: now also C13.1, C14.1, C15.1, IC2.OUT, IC6.VEE, IC6.Y, IC7.VEE, IC7.Y, IC8.VEE, IC8.Y; no longer C10.1, C35.1, C37.1, IC1.OUT, IC10.VEE, IC10.Y, IC12.VEE, IC12.Y, IC13.VEE, IC13.Y
- net -VORP: now also C35.1, C36.1, IC10P.V-, MD6.-5V; no longer C25.1, C27.1, IC5P.V-, MD5.-5V
- net -VPH: now also C25.1, C37.1, C38.1, IC12.-VS, IC13.-VS, R14.2; no longer C15.1, C18.1, C24.1, IC6.-VS, IC7.-VS, R10.2
- net 1_SENSOR: now also IC3.Y3; no longer IC11.Y3
- net 1_SENSOR_EN: now also IC6.A, IC6.B, IC6.C; no longer IC10.A, IC10.B, IC10.C
- net 2_SENSOR: now also IC3.Y0, MD2.OUT; no longer IC11.Y0, MD7.OUT
- net 2_SENSOR_EN: now also IC7.A, IC7.B, IC7.C; no longer IC12.A, IC12.B, IC12.C
- net 3_SENSOR: now also IC3.Y1, MD3.OUT; no longer IC11.Y1, MD8.OUT
- net 3_SENSOR_EN: now also IC8.A, IC8.B, IC8.C; no longer IC13.A, IC13.B, IC13.C
- net A14: now also IC3.Y4; no longer IC11.Y4
- net A15: now also IC3.Y6; no longer IC11.Y6
- net CS_SD: now also IC5A.I; no longer IC4A.I
- net D44: now also IC3.Y5; no longer IC11.Y5
- net D45: now also IC3.Y7; no longer IC11.Y7
- net EC_IN: now also C24.1, IC11.TRE, IC11.TRI, MD5.PR+; no longer C32.1, IC9.TRE, IC9.TRI, MD6.PR+
- net EC_SENSOR: now also IC11.OUT, MD5.OUT, MD5.PR-; no longer IC9.OUT, MD6.OUT, MD6.PR-
- net EN_BAT: now also IC4.EN; no longer IC3.EN
- net FREQ_SENSOR: now also IC3.Z; no longer IC11.Z
- net GND: now also C12.-, C20.2, C6.2, IC10B.IN+, IC13.IN+, IC2.LV, IC3./E, IC3.VEE, IC4.GND, IC5P.VSS, IC6./E, IC6.GND, IC6.Z, IC7./E, IC7.GND, IC7.Z, IC8./E, IC8.Z, MD6.PR-, R3.1, R5.1, R8.2; no longer C12.2, C30.2, C6.-, IC1.LV, IC10./E, IC10.GND, IC10.Z, IC11./E, IC11.VEE, IC12./E, IC12.GND, IC12.Z, IC13./E, IC13.GND, IC13.Z, IC4P.VSS, IC5B.IN+, IC7.IN+, MD5.PR-, R1.1, R13.1, R4.2
- net GSM_KEY: now also IC1.KEY; no longer IC2.KEY
- net GSM_NS: now also IC1.NS; no longer IC2.NS
- net GSM_PT: now also IC1.PS; no longer IC2.PS
- net GSM_RI: now also IC1.RI; no longer IC2.RI
- net GSM_RST: now also IC1.RST; no longer IC2.RST
- net LUZ_SENSOR: now also R5.2; no longer R13.2
- net MOSI: now also IC5B.I; no longer IC4B.I
- net N$10: now also C29.1, IC11.CON; no longer C30.1, IC9.CON
- net N$11: now also MD2.PR-; no longer MD7.PR-
- net N$12: now also MD2.PR+; no longer MD7.PR+
- net N$13: now also MD3.PR-; no longer MD8.PR-
- net N$14: now also IC2.CAP-; no longer IC1.CAP-
- net N$15: now also C27.1, IC10A.IN-, IC10A.OUT; no longer C21.1, IC5A.IN-, IC5A.OUT
- net N$16: now also IC2.CAP+; no longer IC1.CAP+
- net N$17: now also IC10B.IN-, R12.1; no longer IC5B.IN-, R11.1
- net N$18: now also IC4.ADJ, R3.2, R4.2; no longer IC3.ADJ, R1.2, R2.2
- net N$19: now also IC5C.O; no longer IC4C.O
- net N$2: now also C28.1, IC12.IN+, R6.2; no longer C19.1, IC6.IN+, R3.2
- net N$20: now also IC5B.O; no longer IC4B.O
- net N$21: now also IC5A.O; no longer IC4A.O
- net N$22: now also MD3.PR+; no longer MD8.PR+
- net N$23: now also MD5.-5V; no longer MD6.-5V
- net N$24: now also IC6.X0; no longer IC10.X0
- net N$25: now also IC6.Y0; no longer IC10.Y0
- net N$26: now also IC6.Z0; no longer IC10.Z0
- net N$27: now also IC7.Z0, MD2.GND; no longer IC12.Z0, MD7.GND
- net N$28: now also IC7.Y0, MD2.-5V; no longer IC12.Y0, MD7.-5V
- net N$29: now also IC7.X0, MD2.+5V; no longer IC12.X0, MD7.+5V
- net N$3: now also C30.1, IC12.IN-, R10.S; no longer C20.1, IC6.IN-, R5.S
- net N$30: now also IC8.X0, MD3.+5V; no longer IC13.X0, MD8.+5V
- net N$31: now also IC8.Y0, MD3.-5V; no longer IC13.Y0, MD8.-5V
- net N$32: now also IC8.Z0, MD3.GND; no longer IC13.Z0, MD8.GND
- net N$4: now also C30.2, IC12.OUT, R11.2, R13.2; no longer C20.2, IC6.OUT, R6.2, R8.2
- net N$5: now also IC13.IN-, R13.1, R14.1, R15.1; no longer IC7.IN-, R10.1, R12.1, R8.1
- net N$6: now also R10.E, R8.1; no longer R4.1, R5.E
- net N$7: now also C18.1; no longer C16.1
- net N$8: now also R10.A, R11.1; no longer R5.A, R6.1
- net ORP_IN: now also IC10A.IN+, MD6.PR+; no longer IC5A.IN+, MD5.PR+
- net ORP_SENSOR: now also IC10B.OUT, MD6.OUT, R12.2; no longer IC5B.OUT, MD5.OUT, R11.2
- net PH_IN: now also R6.1; no longer R3.1
- net PH_SENSOR: now also IC13.OUT, R15.2; no longer IC7.OUT, R12.2
- net RX2: now also IC1.TX; no longer IC2.TX
- net SCK: now also IC5C.I; no longer IC4C.I
- net SCL: now also IC9.SCK, R1.1; no longer IC8.SCK, R15.1
- net SDA: now also IC9.DATA, R2.1; no longer IC8.DATA, R14.1
- net SELECT_A: now also IC3.A; no longer IC11.A
- net SELECT_B: now also IC3.B; no longer IC11.B
- net SELECT_C: now also IC3.C; no longer IC11.C
- net TX2: now also IC1.RX; no longer IC2.RX
Other:
- moved on the sheet: C10, C11, C13, C14, C15, C16, C17, C18, C19, C20, C21, C22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

Commit message: - Versao enviada para producao
Connections:
- net 1_SENSOR renamed S1_SENSOR
- net 1_SENSOR_EN renamed S1_EN
- net 2_SENSOR renamed S2_SENSOR
- net 2_SENSOR_EN renamed S2_EN
- net 3_SENSOR renamed S3_SENSOR
- net 3_SENSOR_EN renamed S3_EN
- net LUZ_SENSOR renamed LUZ
Other:
- moved on the sheet: C21, C22, C23, C24, C25, C26, C27, C28, C29, C30, C31, C32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
